File: leo65keyboard.sch (KiCad schematic (older format))
At the start: 14 parts

Commit message: finished diagram
Parts:
- added D1, D10, D11, D12, D13, D14, D15, D16, D17, D18, D19, D2, D20, D21, D22, D23, D24, D25, D26, D27, D28, D29, D3, D30, D31, D32, D33, D34, D35, D36, D37, D38, D39, D4, D40, D41, D42, D43, D44, D45, D46, D47, D48, D49, D5, D50, D51, D52, D53, D54, D55, D56, D57, D58, D59, D6, D60, D61, D62, D63, D64, D65, D66, D67, D68, D69, D7, D70, D71, D72, D73, D74, D75, D76, D77, D78, D79, D8, D80, D81, D82, D83, D84, D85, D86, D87, D88, D89, D9, D90: D_Small, MX_Alps_Hybrid:MX-1U-NoLED, symbol Device:D_Small
- added F1: Polyfuse, MX_Alps_Hybrid:MX-1U-NoLED, symbol Device:Polyfuse
- added MX1, MX10, MX11, MX12, MX13, MX14, MX15, MX16, MX17, MX18, MX19, MX2, MX20, MX21, MX22, MX23, MX24, MX25, MX26, MX27, MX28, MX29, MX3, MX30, MX31, MX32, MX33, MX34, MX35, MX36, MX37, MX38, MX39, MX4, MX40, MX41, MX42, MX43, MX44, MX45, MX46, MX47, MX48, MX49, MX5, MX50, MX51, MX52, MX53, MX54, MX55, MX56, MX57, MX58, MX59, MX6, MX60, MX61, MX62, MX63, MX64, MX65, MX66, MX67, MX68, MX69, MX7, MX70, MX71, MX72, MX73, MX74, MX75, MX76, MX77, MX78, MX79, MX8, MX80, MX81, MX82, MX83, MX84, MX85, MX86, MX87, MX88, MX89, MX9, MX90: MX-NoLED, MX_Alps_Hybrid:MX-1U-NoLED, symbol MX_Alps_Hybrid:MX-NoLED
- added USB1: Molex-0548190589, random-keyboard-parts:Molex-0548190589, symbol random-keyboard-parts:Molex-0548190589
- C1, C2, C3, C4, C5, C6, C7: renamed from C?; footprint (none) -> Capacitor_SMD:C_0805_2012Metric_Pad1.15x1.40mm_HandSolder
- R1, R2, R3, R4: renamed from R?; footprint (none) -> Resistor_SMD:R_0805_2012Metric
- SW1: renamed from SW?; footprint (none) -> random-keyboard-parts:SKQG-1155865
- Y1: renamed from Y?; footprint (none) -> Crystal:Crystal_SMD_3225-4Pin_3.2x2.5mm
- gave numbers to parts that had none: 1
Connections:
- net +5V: now also F1.1
- net D+: now also USB1.3 (D+)
- net D-: now also USB1.4 (D-)
- new net: D1.2 (A), MX1.2 (ROW)
- new net: D6.2 (A), MX6.2 (ROW)
- new net: D11.2 (A), MX11.2 (ROW)
- new net: D16.2 (A), MX16.2 (ROW)
- new net: D21.2 (A), MX21.2 (ROW)
- new net: D26.2 (A), MX26.2 (ROW)
- new net: D31.2 (A), MX31.2 (ROW)
- new net: D36.2 (A), MX36.2 (ROW)
- new net: D41.2 (A), MX41.2 (ROW)
- new net: D46.2 (A), MX46.2 (ROW)
- new net: D51.2 (A), MX51.2 (ROW)
- new net: D56.2 (A), MX56.2 (ROW)
- new net: D61.2 (A), MX61.2 (ROW)
- new net: D66.2 (A), MX66.2 (ROW)
- new net: D71.2 (A), MX71.2 (ROW)
- new net: D76.2 (A), MX76.2 (ROW)
- new net: D81.2 (A), MX81.2 (ROW)
- new net: D86.2 (A), MX86.2 (ROW)
- new net: D2.2 (A), MX2.2 (ROW)
- new net: D7.2 (A), MX7.2 (ROW)
- new net: D12.2 (A), MX12.2 (ROW)
- new net: D17.2 (A), MX17.2 (ROW)
- new net: D22.2 (A), MX22.2 (ROW)
- new net: D27.2 (A), MX27.2 (ROW)
- new net: D32.2 (A), MX32.2 (ROW)
- new net: D37.2 (A), MX37.2 (ROW)
- new net: D42.2 (A), MX42.2 (ROW)
- new net: D47.2 (A), MX47.2 (ROW)
- new net: D52.2 (A), MX52.2 (ROW)
- new net: D57.2 (A), MX57.2 (ROW)
- new net: D62.2 (A), MX62.2 (ROW)
- new net: D67.2 (A), MX67.2 (ROW)
- new net: D72.2 (A), MX72.2 (ROW)
- new net: D77.2 (A), MX77.2 (ROW)
- new net: D82.2 (A), MX82.2 (ROW)
- new net: D87.2 (A), MX87.2 (ROW)
- new net: D3.2 (A), MX3.2 (ROW)
- new net: D8.2 (A), MX8.2 (ROW)
- new net: D13.2 (A), MX13.2 (ROW)
- new net: D18.2 (A), MX18.2 (ROW)
- new net: D23.2 (A), MX23.2 (ROW)
- new net: D28.2 (A), MX28.2 (ROW)
- new net: D33.2 (A), MX33.2 (ROW)
- new net: D38.2 (A), MX38.2 (ROW)
- new net: D43.2 (A), MX43.2 (ROW)
- new net: D48.2 (A), MX48.2 (ROW)
- new net: D53.2 (A), MX53.2 (ROW)
- new net: D58.2 (A), MX58.2 (ROW)
- new net: D63.2 (A), MX63.2 (ROW)
- new net: D68.2 (A), MX68.2 (ROW)
- new net: D73.2 (A), MX73.2 (ROW)
- new net: D78.2 (A), MX78.2 (ROW)
- new net: D83.2 (A), MX83.2 (ROW)
- new net: D88.2 (A), MX88.2 (ROW)
- new net: D4.2 (A), MX4.2 (ROW)
- new net: D9.2 (A), MX9.2 (ROW)
- new net: D14.2 (A), MX14.2 (ROW)
- new net: D19.2 (A), MX19.2 (ROW)
- new net: D24.2 (A), MX24.2 (ROW)
- new net: D29.2 (A), MX29.2 (ROW)
- new net: D34.2 (A), MX34.2 (ROW)
- new net: D39.2 (A), MX39.2 (ROW)
- new net: D44.2 (A), MX44.2 (ROW)
- new net: D49.2 (A), MX49.2 (ROW)
- new net: D54.2 (A), MX54.2 (ROW)
- new net: D59.2 (A), MX59.2 (ROW)
- new net: D64.2 (A), MX64.2 (ROW)
- new net: D69.2 (A), MX69.2 (ROW)
- new net: D74.2 (A), MX74.2 (ROW)
- new net: D79.2 (A), MX79.2 (ROW)
- new net: D84.2 (A), MX84.2 (ROW)
- new net: D89.2 (A), MX89.2 (ROW)
- new net: D5.2 (A), MX5.2 (ROW)
- new net: D10.2 (A), MX10.2 (ROW)
- new net: D15.2 (A), MX15.2 (ROW)
- new net: D20.2 (A), MX20.2 (ROW)
- new net: D25.2 (A), MX25.2 (ROW)
- new net: D30.2 (A), MX30.2 (ROW)
- new net: D35.2 (A), MX35.2 (ROW)
- new net: D40.2 (A), MX40.2 (ROW)
- new net: D45.2 (A), MX45.2 (ROW)
- new net: D50.2 (A), MX50.2 (ROW)
- new net: D55.2 (A), MX55.2 (ROW)
- new net: D60.2 (A), MX60.2 (ROW)
- new net: D65.2 (A), MX65.2 (ROW)
- new net: D70.2 (A), MX70.2 (ROW)
- new net: D75.2 (A), MX75.2 (ROW)
- new net: D80.2 (A), MX80.2 (ROW)
- new net: D85.2 (A), MX85.2 (ROW)
- new net: D90.2 (A), MX90.2 (ROW)
- new net Col0: MX1.1 (COL), MX2.1 (COL), MX3.1 (COL), MX4.1 (COL), MX5.1 (COL)
- new net Col1: MX10.1 (COL), MX6.1 (COL), MX7.1 (COL), MX8.1 (COL), MX9.1 (COL)
- new net Col10: MX51.1 (COL), MX52.1 (COL), MX53.1 (COL), MX54.1 (COL), MX55.1 (COL)
- new net Col11: MX56.1 (COL), MX57.1 (COL), MX58.1 (COL), MX59.1 (COL), MX60.1 (COL)
- new net Col12: MX61.1 (COL), MX62.1 (COL), MX63.1 (COL), MX64.1 (COL), MX65.1 (COL)
- new net Col13: MX66.1 (COL), MX67.1 (COL), MX68.1 (COL), MX69.1 (COL), MX70.1 (COL)
- new net Col14: MX71.1 (COL), MX72.1 (COL), MX73.1 (COL), MX74.1 (COL), MX75.1 (COL)
- new net Col15: MX76.1 (COL), MX77.1 (COL), MX78.1 (COL), MX79.1 (COL), MX80.1 (COL)
- new net Col16: MX81.1 (COL), MX82.1 (COL), MX83.1 (COL), MX84.1 (COL), MX85.1 (COL)
- new net Col17: MX86.1 (COL), MX87.1 (COL), MX88.1 (COL), MX89.1 (COL), MX90.1 (COL)
- new net Col2: MX11.1 (COL), MX12.1 (COL), MX13.1 (COL), MX14.1 (COL), MX15.1 (COL)
- new net Col3: MX16.1 (COL), MX17.1 (COL), MX18.1 (COL), MX19.1 (COL), MX20.1 (COL)
- new net Col4: MX21.1 (COL), MX22.1 (COL), MX23.1 (COL), MX24.1 (COL), MX25.1 (COL)
- new net Col5: MX26.1 (COL), MX27.1 (COL), MX28.1 (COL), MX29.1 (COL), MX30.1 (COL)
- new net Col6: MX31.1 (COL), MX32.1 (COL), MX33.1 (COL), MX34.1 (COL), MX35.1 (COL)
- new net Col7: MX36.1 (COL), MX37.1 (COL), MX38.1 (COL), MX39.1 (COL), MX40.1 (COL)
- new net Col8: MX41.1 (COL), MX42.1 (COL), MX43.1 (COL), MX44.1 (COL), MX45.1 (COL)
- new net Col9: MX46.1 (COL), MX47.1 (COL), MX48.1 (COL), MX49.1 (COL), MX50.1 (COL)
- new net Row0: D1.1 (K), D11.1 (K), D16.1 (K), D21.1 (K), D26.1 (K), D31.1 (K), D36.1 (K), D41.1 (K), D46.1 (K), D51.1 (K), D56.1 (K), D6.1 (K), D61.1 (K), D66.1 (K), D71.1 (K), D76.1 (K), D81.1 (K), D86.1 (K)
- new net Row1: D12.1 (K), D17.1 (K), D2.1 (K), D22.1 (K), D27.1 (K), D32.1 (K), D37.1 (K), D42.1 (K), D47.1 (K), D52.1 (K), D57.1 (K), D62.1 (K), D67.1 (K), D7.1 (K), D72.1 (K), D77.1 (K), D82.1 (K), D87.1 (K)
- new net Row2: D13.1 (K), D18.1 (K), D23.1 (K), D28.1 (K), D3.1 (K), D33.1 (K), D38.1 (K), D43.1 (K), D48.1 (K), D53.1 (K), D58.1 (K), D63.1 (K), D68.1 (K), D73.1 (K), D78.1 (K), D8.1 (K), D83.1 (K), D88.1 (K)
- new net Row3: D14.1 (K), D19.1 (K), D24.1 (K), D29.1 (K), D34.1 (K), D39.1 (K), D4.1 (K), D44.1 (K), D49.1 (K), D54.1 (K), D59.1 (K), D64.1 (K), D69.1 (K), D74.1 (K), D79.1 (K), D84.1 (K), D89.1 (K), D9.1 (K)
- new net Row4: D10.1 (K), D15.1 (K), D20.1 (K), D25.1 (K), D30.1 (K), D35.1 (K), D40.1 (K), D45.1 (K), D5.1 (K), D50.1 (K), D55.1 (K), D60.1 (K), D65.1 (K), D70.1 (K), D75.1 (K), D80.1 (K), D85.1 (K), D90.1 (K)
- new net VCC: F1.2, USB1.5 (VBUS)
Other:
- moved on the sheet: C1, C2, C3, C4, C5, C6, C7, R1, R2, R3, R4, SW1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
